Commit message: feat(bonetag_femur):add file tag to urdf filename

File: interfaces/panda_prosthesis/urdf/bonetag_femur.in.urdf (robot description, URDF)
Before this commit: robot bonetag_femur, 3 links, 2 joints
Links:
- link femur: geometry collision mesh filename=file://@DATA_DIR@/meshes/bonetag_femur/femur.stl scale=0.001 0.001 0.001; visual mesh filename=file://@DATA_DIR@/meshes/bonetag_femur/femur.stl scale=0.001 0.001 0.001
- link support_femur: geometry collision mesh filename=file://@DATA_DIR@/meshes/bonetag_femur/support_femur.stl scale=0.001 0.001 0.001; visual mesh filename=file://@DATA_DIR@/meshes/bonetag_femur/support_femur.stl scale=0.001 0.001 0.001
