Commit message: chore: adjust plate module collision box

File: plate/urdf/plate.in.urdf (robot description, URDF)
Before this commit: robot plate, 2 links, 1 joints
Joints:
- removed joint plate_adapter_joint
- added joint plate_joint: type fixed, parent plate_base_link, child plate_link, origin xyz=0.0 0.0 0.0 rpy=0 0 0

Commit message: fix: scale down plate and screw meshes and use them for convex generation

File: plate/urdf/plate.in.urdf (robot description, URDF)
Before this commit: robot plate, 2 links, 1 joints
Links:
- link plate_link: geometry collision mesh filename=file://@MC_MESH_DIR@/plate.stl; visual mesh filename=file://@MC_MESH_DIR@/plate.stl

File: screw/urdf/screw.in.urdf (robot description, URDF)
Before this commit: robot screw, 2 links, 1 joints
Links:
- link screw_link: geometry collision mesh filename=file://@MC_MESH_DIR@/screw.stl scale=0.001 0.001 0.001; visual mesh filename=file://@MC_MESH_DIR@/screw.stl
