Commit message: chore: change name from "camera" to "realsense_camera"

File: realsense_camera/urdf/realsense_d435.in.urdf (robot description, URDF)
Before this commit: robot camera, 3 links, 2 joints
Links:
- removed link bracket_link
- removed link camera_base_link
- removed link camera_link
- added link realsense_d435_base_link
- added link realsense_d435_bracket_link, mass 0.0698; collision mesh filename=file://@MC_MESH_DIR@/realsense_d435_bracket.stl; visual mesh filename=file://@MC_MESH_DIR@/realsense_d435_bracket.stl
- added link realsense_d435_camera_link, mass 0.0698; collision box size=0.09 0.0243 0.0285; visual box size=0.09 0.0243 0.0285
- added link realsense_d435_wrench_link
Joints:
- removed joint camera_joint_1
- removed joint camera_joint_2
- added joint realsense_d435_bracket_joint: type fixed, parent realsense_d435_base_link, child realsense_d435_bracket_link, origin xyz=0.0 0.0 0.0 rpy=0 0 0
- added joint realsense_d435_camera_joint: type fixed, parent realsense_d435_bracket_link, child realsense_d435_camera_link, origin xyz=0.0 0.0 0.0 rpy=0 0 0
- added joint realsense_d435_wrench_joint: type fixed, parent realsense_d435_bracket_link, child realsense_d435_wrench_link, origin xyz=0.0 0.0 0.006 rpy=0 0 0

Commit message: fix: allign all frame with base frame orientation

File: realsense_camera/urdf/realsense_d435.in.urdf (robot description, URDF)
Before this commit: robot realsense_d435, 4 links, 3 joints
Joints:
- joint realsense_d435_bracket_joint: origin xyz=0.0 0.0 0.0 rpy=0 0 0 -> xyz=0.0 0.0 0.0 rpy=0 0 3.14159
