Commit message: modified handE gripper

File: robotiq_gripper/xacro/robotiq_hande_gripper.urdf.xacro (robot description, xacro)
@@ -10,11 +10,15 @@
     <xacro:arg name="slave_id" default="9" />
     <xacro:arg name="frequency_hz" default="10" />
+    <xacro:arg name="grip_pos_min" default="0" />
+    <xacro:arg name="grip_pos_max" default="0.025" />
+    <xacro:arg name="xyz" default="0 0 0" />
+    <xacro:arg name="rpy" default="0 0 0" />
     <!-- Import macros -->
     <xacro:include filename="$(find robotiq_hande_description)/urdf/robotiq_hande_gripper.xacro" />
     <link name="robotiq_hande_origin" />
-    <xacro:robotiq_gripper name="RobotiqGripperHardwareInterface" prefix=""
+    <xacro:robotiq_hande_gripper name="RobotiqGripperHardwareInterface" prefix=""
         parent="robotiq_hande_origin"
-        grip_pos_min="0"
-        grip_pos_max="0.025"
+        grip_pos_min="$(arg grip_pos_min)"
+        grip_pos_max="$(arg grip_pos_max)"
         tty_port="$(arg com_port)"
         baudrate="$(arg baudrate)"
@@ -24,6 +28,7 @@
         slave_id="$(arg slave_id)"
         use_fake_hardware="$(arg use_fake_hardware)"
-        frequency_hz="$(arg frequency_hz)">
-        <origin xyz="0 0 0" rpy="0 0 0" />
-    </xacro:robotiq_gripper>
+        frequency_hz="$(arg frequency_hz)"
+        xyz="$(arg xyz)"
+        rpy="$(arg rpy)">
+    </xacro:robotiq_hande_gripper>
 </robot>
